File: ADS1271_pcb/_saved_ADS1271_pcb.sch (KiCad schematic (older format))
At the start: 2 parts, among them U1 ADS1271

Commit message: Documentación en README
Parts:
- added J?: Conn_01x06_Male, symbol Conn_01x06_Male
Connections:
- net DRBY: now reaches U1.10 (DRBY/FSYNC)
- net SCLK: now reaches U1.11 (SCLK)
- net CLK: now reaches U1.12 (CLK)
- net DVDD: now reaches U1.13 (DVDD)
- net DGND: now reaches U1.14 (DGND)
- net DOUT: now reaches U1.9 (DOUT)
Other:
- note added: "Pines FPGA\n"
Changed lines of the file:
@@
 Wire Wire Line
 	3900 4350 3900 4200
+$Comp
+L Conn_01x06_Male J?
+U 1 1 5B16767B
+P 7400 3050
+F 0 "J?" H 7450 3400 50  0000 C CNN
+F 1 "Conn_01x06_Male" H 7400 2650 50  0000 C CNN
+F 2 "" H 7400 3050 50  0001 C CNN
+F 3 "" H 7400 3050 50  0001 C CNN
+	1    7400 3050
+	1    0    0    -1
+$EndComp
+Text Label 7400 2850 2    60   ~ 0
+DVDD
+Text Label 5250 1900 1    60   ~ 0
+DVDD
+Text Label 7400 2950 2    60   ~ 0
+DGND
+Text Label 5350 4200 3    60   ~ 0
+DGND
+Text Notes 7000 2600 0    79   ~ 0
+Pines FPGA\n
+Text Label 7400 3050 2    61   ~ 0
+DOUT
+Text Label 7400 3150 2    61   ~ 0
+SCLK
+Text Label 7400 3250 2    61   ~ 0
+CLK
+Text Label 7400 3350 2    61   ~ 0
+DRBY
+Text Label 5900 2500 0    61   ~ 0
+DRBY
+Text Label 5900 2800 0    61   ~ 0
+DOUT
+Text Label 5900 3150 0    61   ~ 0
+SCLK
+Text Label 5900 3450 0    61   ~ 0
+CLK
 $EndSCHEMATC

Commit message: Se sume imagen circuito
Parts:
- added R? (x4): R, symbol R
Connections:
- net CLK: no longer U1.12 (CLK)
- net DOUT: no longer U1.9 (DOUT)
- net DRBY: no longer U1.10 (DRBY/FSYNC)
- net SCLK: no longer U1.11 (SCLK)
Changed lines of the file:
@@
 Text Label 7400 3350 2    61   ~ 0
 DRBY
-Text Label 5900 2500 0    61   ~ 0
+Text Label 6350 2500 0    61   ~ 0
 DRBY
-Text Label 5900 2800 0    61   ~ 0
+Text Label 6350 2800 0    61   ~ 0
 DOUT
-Text Label 5900 3150 0    61   ~ 0
+Text Label 6350 3150 0    61   ~ 0
 SCLK
-Text Label 5900 3450 0    61   ~ 0
+Text Label 6350 3450 0    61   ~ 0
 CLK
+$Comp
+L R R?
+U 1 1 5B167FA3
+P 6100 2500
+F 0 "R?" V 6180 2500 50  0000 C CNN
+F 1 "R" V 6100 2500 50  0000 C CNN
+F 2 "" V 6030 2500 50  0001 C CNN
+F 3 "" H 6100 2500 50  0001 C CNN
+	1    6100 2500
+	0    1    1    0
+$EndComp
+$Comp
+L R R?
+U 1 1 5B167FD4
+P 6100 2800
+F 0 "R?" V 6180 2800 50  0000 C CNN
+F 1 "R" V 6100 2800 50  0000 C CNN
+F 2 "" V 6030 2800 50  0001 C CNN
+F 3 "" H 6100 2800 50  0001 C CNN
+	1    6100 2800
+	0    1    1    0
+$EndComp
+$Comp
+L R R?
+U 1 1 5B1680B7
+P 6100 3150
+F 0 "R?" V 6180 3150 50  0000 C CNN
+F 1 "R" V 6100 3150 50  0000 C CNN
+F 2 "" V 6030 3150 50  0001 C CNN
+F 3 "" H 6100 3150 50  0001 C CNN
+	1    6100 3150
+	0    1    1    0
+$EndComp
+$Comp
+L R R?
+U 1 1 5B1680E5
+P 6100 3450
+F 0 "R?" V 6180 3450 50  0000 C CNN
+F 1 "R" V 6100 3450 50  0000 C CNN
+F 2 "" V 6030 3450 50  0001 C CNN
+F 3 "" H 6100 3450 50  0001 C CNN
+	1    6100 3450
+	0    1    1    0
+$EndComp
 $EndSCHEMATC
