File: ADS1271_pcb/ADS1271_pcb.kicad_pcb (KiCad board)
At the start: 2 copper layers, 1 part, among them U1 ADS1271

Commit message: PCB Terminado
Parts:
- added C1: 0.33 uf, Capacitors_THT:CP_Radial_D5.0mm_P2.50mm, F.Cu at (108.5, 122.2)
- added C2: 0,1 uf, Capacitors_THT:CP_Radial_D5.0mm_P2.50mm, F.Cu at (109.6, 114.2)
- added C3: 100pF, Capacitors_THT:C_Disc_D5.0mm_W2.5mm_P5.00mm, F.Cu at (109.0, 103.4)
- added C4: 100pF, Capacitors_THT:C_Disc_D5.0mm_W2.5mm_P5.00mm, F.Cu at (109.0, 99.0)
- added C5: 1nF, Capacitors_THT:C_Disc_D5.0mm_W2.5mm_P5.00mm, F.Cu at (104.2, 107.6)
- added C6: 10 uf, Capacitors_THT:CP_Radial_D5.0mm_P2.50mm, F.Cu at (134.2, 123.1)
- added C7: 10uF, Capacitors_THT:CP_Radial_D5.0mm_P2.50mm, F.Cu at (126.8, 99.0)
- added C8: 100nF, Capacitors_THT:CP_Radial_D5.0mm_P2.50mm, F.Cu at (131.6, 113.2)
- added J1: conector +7V, Connectors_Molex:Molex_SPOX-5267_22-03-5025_02x2.54mm_Straight, F.Cu at (99.5, 123.5)
- added J2: CONN_01X02_ent_dif, Connectors_Molex:Molex_SPOX-5267_22-03-5025_02x2.54mm_Straight, F.Cu at (91.0, 100.0)
- added J3: Conn_01x06_Male_fpga_pins, Connectors_Molex:Molex_SPOX-5267_22-03-5065_06x2.54mm_Straight, F.Cu at (157.3, 109.0)
- added JP1: Jumper_NC_Dual_selec_modo, Connectors_Molex:Molex_SPOX-5267_22-03-5035_03x2.54mm_Straight, F.Cu at (126.2, 88.5)
- added R1: 680, Resistors_THT:R_Axial_DIN0207_L6.3mm_D2.5mm_P5.08mm_Vertical, F.Cu at (145.7, 120.4)
- added R2: 50, Resistors_THT:R_Axial_DIN0207_L6.3mm_D2.5mm_P5.08mm_Vertical, F.Cu at (119.8, 98.5)
- added R3: 50, Resistors_THT:R_Axial_DIN0207_L6.3mm_D2.5mm_P5.08mm_Vertical, F.Cu at (139.0, 99.8)
- added R4: 50, Resistors_THT:R_Axial_DIN0207_L6.3mm_D2.5mm_P5.08mm_Vertical, F.Cu at (139.0, 95.9)
- added R5: 50, Resistors_THT:R_Axial_DIN0207_L6.3mm_D2.5mm_P5.08mm_Vertical, F.Cu at (138.9, 103.5)
- added R6: 50, Resistors_THT:R_Axial_DIN0207_L6.3mm_D2.5mm_P5.08mm_Vertical, F.Cu at (138.9, 107.2)
- added U2: LM336z2.5, TO_SOT_Packages_THT:TO-92_Inline_Narrow_Oval, F.Cu at (126.5, 117.0)
- added U3: ADS1271, Housings_SSOP:TSSOP-16_4.4x5mm_Pitch0.65mm, B.Cu at (120.4, 107.1)
- U1: value ADS1271 -> LM7805_us; footprint Housings_SSOP:TSSOP-16_4.4x5mm_Pitch0.65mm -> TO_SOT_Packages_THT:TO-220-3_Vertical
- moved U1 54.8 mm to (95.0, 117.0), turned to 90 degrees
Connections:
- U1 pad 2: Net-(U1-Pad2) -> GNDA
Routing:
- net /DVDD: track 0.00 -> 95.9 mm
- net Net-(JP1-Pad2): track 0.00 -> 35.5 mm
- net Net-(C4-Pad2): track 0.00 -> 34.5 mm
- net Net-(C6-Pad1): track 0.00 -> 33.4 mm
- net Net-(C3-Pad2): track 0.00 -> 33.4 mm
- net Net-(C2-Pad1): track 0.00 -> 31.7 mm
- net /DRBY: track 0.00 -> 30.7 mm
- net /DGND: track 0.00 -> 27.9 mm
- net /DOUT: track 0.00 -> 20.7 mm
- net /SCLK: track 0.00 -> 19.4 mm
- net /CLK: track 0.00 -> 18.7 mm
- net Net-(C1-Pad1): track 0.00 -> 18.5 mm
- net Net-(R4-Pad2): track 0.00 -> 15.1 mm
- net Net-(R3-Pad2): track 0.00 -> 12.9 mm
- net Net-(R5-Pad2): track 0.00 -> 11.6 mm
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- added copper zone on B.Cu, net /DGND
- added copper zone on B.Cu, net GNDA
Other:
- rule pad_to_mask_clearance: 0.2 -> 0
- board text added: "AVDD AGND"
- board text added: "DVDD DGND DOUT SCLK CLK DRBY"
- board text added: "ENTRADA DIFERENCIAL"
- board text added: "REFERENCIA ANALÓGICA"
- board text added: "salida Pmod zedboard"

Commit message: Se cambian dos capacitores de ceramica por dos electroliticos, en entrada dvdd (pin 13)
Parts:
- C7: value 10uF -> 10 uf
- C8: value 100nF -> 0.1 uF
- moved C8 1.50 mm to (132.5, 112.0), turned to 180 degrees
Connections:
- C7 pad 1: /DGND -> /DVDD
- C7 pad 2: /DVDD -> /DGND
- C8 pad 1: /DGND -> /DVDD
- C8 pad 2: /DVDD -> /DGND
Routing:
- net /DGND: track 27.9 -> 20.5 mm
- net /DVDD: track 95.9 -> 94.9 mm
Changed lines of the file:
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@@
     (links 44)
     (no_connects 0)
-    (area 73.22143 71.3 162.000001 128.385)
+    (area 0 0 0 0)
     (thickness 1.6)
     (drawings 7)
-    (tracks 119)
+    (tracks 116)
     (zones 0)
     (modules 21)
@@
       (effects (font (size 1 1) (thickness 0.15)))
     )
-    (fp_text value 10uF (at 1.25 3.81 270) (layer F.Fab)
+    (fp_text value "10 uf" (at 1.25 3.81 270) (layer F.Fab)
       (effects (font (size 1 1) (thickness 0.15)))
     )
@@
     )
     (pad 1 thru_hole rect (at 0 0 270) (size 1.6 1.6) (drill 0.8) (layers *.Cu *.Mask)
+      (net 8 /DVDD))
+    (pad 2 thru_hole circle (at 2.5 0 270) (size 1.6 1.6) (drill 0.8) (layers *.Cu *.Mask)
       (net 7 /DGND))
-    (pad 2 thru_hole circle (at 2.5 0 270) (size 1.6 1.6) (drill 0.8) (layers *.Cu *.Mask)
-      (net 8 /DVDD))
     (model ${KISYS3DMOD}/Capacitors_THT.3dshapes/CP_Radial_D5.0mm_P2.50mm.wrl
       (at (xyz 0 0 0))
@@
   )
   (module Capacitors_THT:CP_Radial_D5.0mm_P2.50mm (layer F.Cu)
-    (at 131.6 113.2)
+    (at 132.5 112 180)
     (descr "CP, Radial series, Radial, pin pitch=2.50mm, , diameter=5mm, Electrolytic Capacitor")
     (tags "CP Radial series Radial pin pitch 2.50mm  diameter 5mm Electrolytic Capacitor")
-    (fp_text reference C8 (at 1.25 -3.81) (layer F.SilkS)
-      (effects (font (size 1 1) (thickness 0.15)))
-    )
-    (fp_text value 100nF (at 1.25 3.81) (layer F.Fab)
+    (fp_text reference C8 (at 1.25 -3.81 180) (layer F.SilkS)
+      (effects (font (size 1 1) (thickness 0.15)))
+    )
+    (fp_text value "0.1 uF" (at 1.25 3.81 180) (layer F.Fab)
       (effects (font (size 1 1) (thickness 0.15)))
     )
@@
     (fp_line (start 4.1 2.85) (end 4.1 -2.85) (layer F.CrtYd) (width 0.05))
     (fp_line (start 4.1 -2.85) (end -1.6 -2.85) (layer F.CrtYd) (width 0.05))
-    (fp_text user %R (at 1.25 0) (layer F.Fab)
-      (effects (font (size 1 1) (thickness 0.15)))
-    )
-    (pad 1 thru_hole rect (at 0 0) (size 1.6 1.6) (drill 0.8) (layers *.Cu *.Mask)
+    (fp_text user %R (at 1.25 0 180) (layer F.Fab)
+      (effects (font (size 1 1) (thickness 0.15)))
+    )
+    (pad 1 thru_hole rect (at 0 0 180) (size 1.6 1.6) (drill 0.8) (layers *.Cu *.Mask)
+      (net 8 /DVDD))
+    (pad 2 thru_hole circle (at 2.5 0 180) (size 1.6 1.6) (drill 0.8) (layers *.Cu *.Mask)
       (net 7 /DGND))
-    (pad 2 thru_hole circle (at 2.5 0) (size 1.6 1.6) (drill 0.8) (layers *.Cu *.Mask)
-      (net 8 /DVDD))
     (model ${KISYS3DMOD}/Capacitors_THT.3dshapes/CP_Radial_D5.0mm_P2.50mm.wrl
       (at (xyz 0 0 0))
@@
   (segment (start 134.2 123.1) (end 143 123.1) (width 0.25) (layer B.Cu) (net 6))
   (segment (start 143 123.1) (end 145.7 120.4) (width 0.25) (layer B.Cu) (net 6))
-  (segment (start 127.1 108.7) (end 131.6 113.2) (width 0.25) (layer B.Cu) (net 7))
-  (segment (start 123.35 108.725) (end 127.125 108.725) (width 0.25) (layer B.Cu) (net 7))
-  (segment (start 127.125 108.725) (end 127.1 108.7) (width 0.25) (layer B.Cu) (net 7))
-  (segment (start 123.35 108.075) (end 126.475 108.075) (width 0.25) (layer B.Cu) (net 7))
-  (segment (start 126.475 108.075) (end 127.1 108.7) (width 0.25) (layer B.Cu) (net 7))
+  (segment (start 123.35 108.725) (end 126.725 108.725) (width 0.25) (layer B.Cu) (net 7) (status 400000))
+  (segment (start 126.725 108.725) (end 126.5 108.5) (width 0.25) (layer B.Cu) (net 7))
+  (segment (start 123.35 108.075) (end 126.075 108.075) (width 0.25) (layer B.Cu) (net 7) (status 400000))
+  (segment (start 126.075 108.075) (end 126.5 108.5) (width 0.25) (layer B.Cu) (net 7))
+  (segment (start 126.5 108.5) (end 130 112) (width 0.25) (layer B.Cu) (net 7) (status 800000))
   (segment (start 121.775 108.725) (end 121.575 108.525) (width 0.25) (layer B.Cu) (net 7))
   (segment (start 121.575 108.525) (end 121.575 108.075) (width 0.25) (layer B.Cu) (net 7))
   (segment (start 123.35 108.725) (end 121.775 108.725) (width 0.25) (layer B.Cu) (net 7))
-  (segment (start 117.45 106.125) (end 120.375 106.125) (width 0.25) (layer B.Cu) (net 7))
   (segment (start 121.575 108.075) (end 123.35 108.075) (width 0.25) (layer B.Cu) (net 7))
-  (segment (start 120.75 107.25) (end 121.575 108.075) (width 0.25) (layer B.Cu) (net 7))
-  (segment (start 120.75 106.5) (end 120.75 107.25) (width 0.25) (layer B.Cu) (net 7))
-  (segment (start 120.375 106.125) (end 120.75 106.5) (width 0.25) (layer B.Cu) (net 7))
   (segment (start 117.45 104.825) (end 116.175 104.825) (width 0.25) (layer B.Cu) (net 7))
   (segment (start 116.125 106.125) (end 117.45 106.125) (width 0.25) (layer B.Cu) (net 7))
@@
   (segment (start 115.75 105.25) (end 115.75 105.75) (width 0.25) (layer B.Cu) (net 7))
   (segment (start 116.175 104.825) (end 115.75 105.25) (width 0.25) (layer B.Cu) (net 7))
+  (segment (start 126.75 101.5) (end 126.5 101.5) (width 0.25) (layer B.Cu) (net 7))
+  (segment (start 132.5 112) (end 142.38 112) (width 0.25) (layer B.Cu) (net 8))
+  (segment (start 142.38 112) (end 145.7 115.32) (width 0.25) (layer B.Cu) (net 8))
+  (segment (start 123.35 107.425) (end 129.725 107.425) (width 0.25) (layer B.Cu) (net 8))
+  (segment (start 132.5 110.2) (end 132.5 112) (width 0.25) (layer B.Cu) (net 8))
+  (segment (start 129.725 107.425) (end 132.5 110.2) (width 0.25) (layer B.Cu) (net 8))
+  (segment (start 124.5 99) (end 122 101.5) (width 0.25) (layer B.Cu) (net 8))
+  (segment (start 122.425 107.425) (end 123.35 107.425) (width 0.25) (layer B.Cu) (net 8))
+  (segment (start 121.5 106.5) (end 122.425 107.425) (width 0.25) (layer B.Cu) (net 8))
+  (segment (start 121.5 102) (end 121.5 106.5) (width 0.25) (layer B.Cu) (net 8))
+  (segment (start 122 101.5) (end 121.5 102) (width 0.25) (layer B.Cu) (net 8))
+  (segment (start 119.75 93.42) (end 119.75 94.25) (width 0.25) (layer B.Cu) (net 8))
+  (segment (start 124.5 99) (end 126.75 99) (width 0.25) (layer B.Cu) (net 8))
+  (segment (start 119.75 94.25) (end 124.5 99) (width 0.25) (layer B.Cu) (net 8))
   (segment (start 131.33 88.5) (end 131.33 89.92) (width 0.25) (layer B.Cu) (net 8))
   (segment (start 131.33 89.92) (end 127.83 93.42) (width 0.25) (layer B.Cu) (net 8))
   (segment (start 127.83 93.42) (end 119.75 93.42) (width 0.25) (layer B.Cu) (net 8))
-  (segment (start 126.75 101.5) (end 126.5 101.5) (width 0.25) (layer B.Cu) (net 8))
-  (segment (start 126.5 101.5) (end 119.75 94.75) (width 0.25) (layer B.Cu) (net 8))
-  (segment (start 119.75 94.75) (end 119.75 93.42) (width 0.25) (layer B.Cu) (net 8))
-  (segment (start 126.75 101.5) (end 125 101.5) (width 0.25) (layer B.Cu) (net 8))
-  (segment (start 121.925 107.425) (end 123.35 107.425) (width 0.25) (layer B.Cu) (net 8))
-  (segment (start 125 101.5) (end 121.5 105) (width 0.25) (layer B.Cu) (net 8))
-  (segment (start 121.5 105) (end 121.5 107) (width 0.25) (layer B.Cu) (net 8))
-  (segment (start 121.5 107) (end 121.925 107.425) (width 0.25) (layer B.Cu) (net 8))
   (segment (start 157.3 96.3) (end 158.3 96.3) (width 0.25) (layer B.Cu) (net 8))
   (segment (start 158.3 96.3) (end 160.25 98.25) (width 0.25) (layer B.Cu) (net 8))
+  (segment (start 155.43 115.32) (end 145.7 115.32) (width 0.25) (layer B.Cu) (net 8))
+  (segment (start 160.25 110.5) (end 155.43 115.32) (width 0.25) (layer B.Cu) (net 8))
   (segment (start 160.25 98.25) (end 160.25 110.5) (width 0.25) (layer B.Cu) (net 8))
-  (segment (start 160.25 110.5) (end 155.43 115.32) (width 0.25) (layer B.Cu) (net 8))
-  (segment (start 155.43 115.32) (end 145.7 115.32) (width 0.25) (layer B.Cu) (net 8))
-  (segment (start 123.35 107.425) (end 129.925 107.425) (width 0.25) (layer B.Cu) (net 8))
-  (segment (start 134.1 111.6) (end 134.1 113.2) (width 0.25) (layer B.Cu) (net 8))
-  (segment (start 129.925 107.425) (end 134.1 111.6) (width 0.25) (layer B.Cu) (net 8))
-  (segment (start 134.1 113.2) (end 143.58 113.2) (width 0.25) (layer B.Cu) (net 8))
-  (segment (start 143.58 113.2) (end 145.7 115.32) (width 0.25) (layer B.Cu) (net 8))
   (segment (start 119.58 93.25) (end 119.75 93.42) (width 0.25) (layer B.Cu) (net 8))
   (segment (start 119.58 92.84) (end 119.5 92.92) (width 0.25) (layer B.Cu) (net 8))
@@
     (polygon
       (pts
-        (xy 162 127) (xy 121 127) (xy 121 107) (xy 114 107) (xy 114 85)
+        (xy 162 127) (xy 120.5 127) (xy 120.5 107) (xy 114 107) (xy 114 85)
         (xy 162 85)
       )
